File: VERA-MODULE-RBL.kicad_pcb (KiCad board)
At the start: 2 copper layers, 0.9 x 0.6 mm, 41 parts, among them J4 DX07S016JA1R1500, Q1 BSS138, Q2 BSS138, Q3 BC817, Q4 BC817, U1 TXB0108DQSR, U10 W25Q16JVSNIQ, U11 WM8524CGEDT, U12 AMS1117-3.3, U13 TLV71325PDBV, U14 CH340T, U2 ICE40UP5K-SG48ITR, U3 TXB0108DQSR, U4 TXB0108DQSR, U8 74CBTLV3126PW,118, X1 SG-5032CAN

Commit message: Updated
Parts:
- added C13: 10uF, Capacitor_SMD:C_1206_3216Metric_Pad1.33x1.80mm_HandSolder, F.Cu at (112.0, 299.3)
- added C14: 100nF, Capacitor_SMD:C_1206_3216Metric_Pad1.33x1.80mm_HandSolder, F.Cu at (118.0, 295.9)
- added C15: 10uF, Capacitor_SMD:C_1206_3216Metric_Pad1.33x1.80mm_HandSolder, F.Cu at (112.0, 302.6)
- added C16: 100nF, Capacitor_SMD:C_1206_3216Metric_Pad1.33x1.80mm_HandSolder, F.Cu at (118.0, 299.3)
- added C17: 10uF, Capacitor_SMD:C_1206_3216Metric_Pad1.33x1.80mm_HandSolder, F.Cu at (112.0, 295.9)
- added C18: 100nF, Capacitor_SMD:C_1206_3216Metric_Pad1.33x1.80mm_HandSolder, F.Cu at (124.0, 295.9)
- added C19: 10uF, Capacitor_SMD:C_1206_3216Metric_Pad1.33x1.80mm_HandSolder, F.Cu at (112.0, 306.0)
- added C20: 100nF, Capacitor_SMD:C_1206_3216Metric_Pad1.33x1.80mm_HandSolder, F.Cu at (118.0, 302.6)
- added C21: 10uF, Capacitor_SMD:C_1206_3216Metric_Pad1.33x1.80mm_HandSolder, F.Cu at (124.0, 299.3)
- added C22: 100nF, Capacitor_SMD:C_1206_3216Metric_Pad1.33x1.80mm_HandSolder, F.Cu at (130.0, 295.9)
- added C23: 100nF, Capacitor_SMD:C_1206_3216Metric_Pad1.33x1.80mm_HandSolder, F.Cu at (118.0, 306.0)
- added C24: 10uF, Capacitor_SMD:C_1206_3216Metric_Pad1.33x1.80mm_HandSolder, F.Cu at (124.0, 302.6)
- added C25: 100nF, Capacitor_SMD:C_1206_3216Metric_Pad1.33x1.80mm_HandSolder, F.Cu at (129.9, 224.9)
- added C26: 4.7uF, Capacitor_SMD:C_1206_3216Metric_Pad1.33x1.80mm_HandSolder, F.Cu at (52.8, 279.1)
- added C27: 100nF, Capacitor_SMD:C_1206_3216Metric_Pad1.33x1.80mm_HandSolder, F.Cu at (64.8, 278.8)
- added C28: 100nF, Capacitor_SMD:C_1206_3216Metric_Pad1.33x1.80mm_HandSolder, F.Cu at (58.8, 282.5)
- added C29: 100nF, Capacitor_SMD:C_1206_3216Metric_Pad1.33x1.80mm_HandSolder, F.Cu at (67.2, 272.1)
- added C30: 1uF, Capacitor_SMD:C_1206_3216Metric_Pad1.33x1.80mm_HandSolder, F.Cu at (71.9, 265.5)
- added C31: 1uF, Capacitor_SMD:C_1206_3216Metric_Pad1.33x1.80mm_HandSolder, F.Cu at (61.2, 275.4)
- added C32: 1uF, Capacitor_SMD:C_1206_3216Metric_Pad1.33x1.80mm_HandSolder, F.Cu at (58.8, 279.1)
- added C33: 1uF, Capacitor_SMD:C_1206_3216Metric_Pad1.33x1.80mm_HandSolder, F.Cu at (61.2, 272.1)
- added C34: 4.7uF, Capacitor_SMD:C_1206_3216Metric_Pad1.33x1.80mm_HandSolder, F.Cu at (52.8, 282.5)
- added C35: 4.7uF, Capacitor_SMD:C_1206_3216Metric_Pad1.33x1.80mm_HandSolder, F.Cu at (67.2, 275.4)
- added C36: 2.2uF, Capacitor_SMD:C_1206_3216Metric_Pad1.33x1.80mm_HandSolder, F.Cu at (71.9, 262.1)
- added C39: 22pF, Capacitor_SMD:C_1206_3216Metric_Pad1.33x1.80mm_HandSolder, F.Cu at (83.6, 236.5)
- added C47: 10uF-35V, Capacitor_Tantalum_SMD:CP_EIA-3528-12_Kemet-T_Pad1.50x2.35mm_HandSolder, F.Cu at (51.4, 251.4)
- added C48: 10uF-20V, Capacitor_Tantalum_SMD:CP_EIA-3528-12_Kemet-T_Pad1.50x2.35mm_HandSolder, F.Cu at (57.7, 251.4)
- added C50: 100nF, Capacitor_SMD:C_1206_3216Metric_Pad1.33x1.80mm_HandSolder, F.Cu at (42.4, 255.2)
- added C51: 10uF-20V, Capacitor_Tantalum_SMD:CP_EIA-3528-12_Kemet-T_Pad1.50x2.35mm_HandSolder, F.Cu at (73.3, 241.7)
- added C52: 100nF, Capacitor_SMD:C_1206_3216Metric_Pad1.33x1.80mm_HandSolder, F.Cu at (63.1, 268.7)
- added C53: 100nF, Capacitor_SMD:C_1206_3216Metric_Pad1.33x1.80mm_HandSolder, F.Cu at (165.1, 253.7)
- added C54: 100nF, Capacitor_SMD:C_1206_3216Metric_Pad1.33x1.80mm_HandSolder, F.Cu at (118.7, 288.9)
- added CART1: ATARI-CARTRIDGE, RetroBitLab:ATARI-LEFT-CARTRIDGE, F.Cu at (207.0, 196.4)
- added ECI1: ECIBUS, RetroBitLab:ATARI-XE-ECI-SLOT, F.Cu at (165.3, 209.8)
- added J1: CONN_SMD_02x08_Odd_Even_2.54mm, Connector_PinHeader_2.54mm:PinHeader_2x08_P2.54mm_Vertical_SMD, F.Cu at (155.7, 263.2)
- added J2: ICD15S13E4GX00LF, RetroBitLab:CONN_DB15_F_AMPHENOL_ICD15S13E4GX00LF, F.Cu at (125.2, 257.5)
- added J3: CONN_DM3AT-SF-PEJM5, RetroBitLab:HRS_DM3AT-SF-PEJM5, F.Cu at (41.5, 270.8)
- added J5: PJ-002AH-SMT-TR, RetroBitLab:CUI_PJ-002AH-SMT-TR, F.Cu at (45.2, 232.4)
- added JP1: Jumper3_Bridged12, Jumper:SolderJumper-3_P1.3mm_Open_RoundedPad1.0x1.5mm, F.Cu at (129.9, 299.4)
- added JP2: Jumper_2_Open, Connector_PinHeader_2.54mm:PinHeader_1x02_P2.54mm_Vertical, F.Cu at (184.1, 268.5)
- added LD1: RED, LED_SMD:LED_1206_3216Metric_Pad1.42x1.75mm_HandSolder, F.Cu at (129.9, 228.3)
- added LD2: GREEN, LED_SMD:LED_1206_3216Metric_Pad1.42x1.75mm_HandSolder, F.Cu at (124.7, 287.5)
- added LD3: RED, LED_SMD:LED_1206_3216Metric_Pad1.42x1.75mm_HandSolder, F.Cu at (141.2, 299.3)
- added LD4: GREEN, LED_SMD:LED_1206_3216Metric_Pad1.42x1.75mm_HandSolder, F.Cu at (141.2, 295.9)
- added R1: 2K7, Resistor_SMD:R_1206_3216Metric_Pad1.30x1.75mm_HandSolder, F.Cu at (165.1, 260.3)
- added R10: 4K3, Resistor_SMD:R_1206_3216Metric_Pad1.30x1.75mm_HandSolder, F.Cu at (161.0, 279.4)
- added R11: 2K, Resistor_SMD:R_1206_3216Metric_Pad1.30x1.75mm_HandSolder, F.Cu at (171.0, 260.3)
- added R12: 150R, Resistor_SMD:R_1206_3216Metric_Pad1.30x1.75mm_HandSolder, F.Cu at (165.1, 266.9)
- added R13: 2K, Resistor_SMD:R_1206_3216Metric_Pad1.30x1.75mm_HandSolder, F.Cu at (148.5, 284.1)
- added R14: 150R, Resistor_SMD:R_1206_3216Metric_Pad1.30x1.75mm_HandSolder, F.Cu at (165.1, 270.2)
- added R15: 2K, Resistor_SMD:R_1206_3216Metric_Pad1.30x1.75mm_HandSolder, F.Cu at (171.0, 263.6)
- added R16: 150R, Resistor_SMD:R_1206_3216Metric_Pad1.30x1.75mm_HandSolder, F.Cu at (166.9, 273.4)
- added R17: 910R, Resistor_SMD:R_1206_3216Metric_Pad1.30x1.75mm_HandSolder, F.Cu at (171.0, 266.9)
- added R18: 160R, Resistor_SMD:R_1206_3216Metric_Pad1.30x1.75mm_HandSolder, F.Cu at (171.0, 270.2)
- added R19: 910R, Resistor_SMD:R_1206_3216Metric_Pad1.30x1.75mm_HandSolder, F.Cu at (154.4, 284.1)
- added R2: 10K, Resistor_SMD:R_1206_3216Metric_Pad1.30x1.75mm_HandSolder, F.Cu at (171.0, 257.0)
- added R20: 160R, Resistor_SMD:R_1206_3216Metric_Pad1.30x1.75mm_HandSolder, F.Cu at (136.6, 287.4)
- added R21: 910R, Resistor_SMD:R_1206_3216Metric_Pad1.30x1.75mm_HandSolder, F.Cu at (161.0, 282.7)
- added R22: 160R, Resistor_SMD:R_1206_3216Metric_Pad1.30x1.75mm_HandSolder, F.Cu at (154.4, 287.4)
- added R23: 510R, Resistor_SMD:R_1206_3216Metric_Pad1.30x1.75mm_HandSolder, F.Cu at (166.9, 276.7)
- added R24: 27R, Resistor_SMD:R_1206_3216Metric_Pad1.30x1.75mm_HandSolder, F.Cu at (172.9, 273.4)
- added R25: 510R, Resistor_SMD:R_1206_3216Metric_Pad1.30x1.75mm_HandSolder, F.Cu at (141.4, 280.8)
- added R26: 27R, Resistor_SMD:R_1206_3216Metric_Pad1.30x1.75mm_HandSolder, F.Cu at (166.9, 280.0)
- added R27: 510R, Resistor_SMD:R_1206_3216Metric_Pad1.30x1.75mm_HandSolder, F.Cu at (129.5, 280.8)
- added R28: 27R, Resistor_SMD:R_1206_3216Metric_Pad1.30x1.75mm_HandSolder, F.Cu at (130.6, 287.5)
- added R29: 820R, Resistor_SMD:R_1206_3216Metric_Pad1.30x1.75mm_HandSolder, F.Cu at (141.5, 277.5)
- added R3: 50R, Resistor_SMD:R_1206_3216Metric_Pad1.30x1.75mm_HandSolder, F.Cu at (165.1, 257.0)
- added R30: 820R, Resistor_SMD:R_1206_3216Metric_Pad1.30x1.75mm_HandSolder, F.Cu at (135.4, 280.8)
- added R31: 4K7, Resistor_SMD:R_1206_3216Metric_Pad1.30x1.75mm_HandSolder, F.Cu at (121.6, 234.9)
- added R32: 330R, Resistor_SMD:R_1206_3216Metric_Pad1.30x1.75mm_HandSolder, F.Cu at (115.5, 241.6)
- added R33: 3K3, Resistor_SMD:R_1206_3216Metric_Pad1.30x1.75mm_HandSolder, F.Cu at (121.6, 238.2)
- added R34: 10K, Resistor_SMD:R_1206_3216Metric_Pad1.30x1.75mm_HandSolder, F.Cu at (127.6, 231.6)
- added R35: 2K7, Resistor_SMD:R_1206_3216Metric_Pad1.30x1.75mm_HandSolder, B.Cu at (172.5, 193.9)
- added R36: 2K7, Resistor_SMD:R_1206_3216Metric_Pad1.30x1.75mm_HandSolder, B.Cu at (176.1, 193.9)
- added R37: 47K, Resistor_SMD:R_1206_3216Metric_Pad1.30x1.75mm_HandSolder, F.Cu at (64.8, 282.1)
- added R38: 47K, Resistor_SMD:R_1206_3216Metric_Pad1.30x1.75mm_HandSolder, F.Cu at (73.2, 272.1)
- added R39: 47K, Resistor_SMD:R_1206_3216Metric_Pad1.30x1.75mm_HandSolder, F.Cu at (70.8, 278.7)
- added R4: 50R, Resistor_SMD:R_1206_3216Metric_Pad1.30x1.75mm_HandSolder, F.Cu at (161.0, 276.1)
- added R40: 47K, Resistor_SMD:R_1206_3216Metric_Pad1.30x1.75mm_HandSolder, F.Cu at (73.2, 275.4)
- added R41: 47K, Resistor_SMD:R_1206_3216Metric_Pad1.30x1.75mm_HandSolder, F.Cu at (64.8, 285.4)
- added R42: 47K, Resistor_SMD:R_1206_3216Metric_Pad1.30x1.75mm_HandSolder, F.Cu at (189.4, 267.9)
- added R43: 47K, Resistor_SMD:R_1206_3216Metric_Pad1.30x1.75mm_HandSolder, F.Cu at (73.2, 268.8)
- added R44: 47K, Resistor_SMD:R_1206_3216Metric_Pad1.30x1.75mm_HandSolder, F.Cu at (70.7, 285.4)
- added R45: 560R, Resistor_SMD:R_1206_3216Metric_Pad1.30x1.75mm_HandSolder, F.Cu at (76.7, 278.7)
- added R46: 560R, Resistor_SMD:R_1206_3216Metric_Pad1.30x1.75mm_HandSolder, F.Cu at (70.7, 282.1)
- added R47: 10K, Resistor_SMD:R_1206_3216Metric_Pad1.30x1.75mm_HandSolder, F.Cu at (72.3, 252.2)
- added R48: 10K, Resistor_SMD:R_1206_3216Metric_Pad1.30x1.75mm_HandSolder, F.Cu at (85.4, 239.8)
- added R49: DNP, Resistor_SMD:R_1206_3216Metric_Pad1.30x1.75mm_HandSolder, F.Cu at (147.1, 295.9)
- added R5: 10K, Resistor_SMD:R_1206_3216Metric_Pad1.30x1.75mm_HandSolder, F.Cu at (135.5, 284.1)
- added R50: 5K1, Resistor_SMD:R_1206_3216Metric_Pad1.30x1.75mm_HandSolder, F.Cu at (89.6, 236.4)
- added R51: 5K1, Resistor_SMD:R_1206_3216Metric_Pad1.30x1.75mm_HandSolder, F.Cu at (75.9, 248.8)
- added R52: 2K2, Resistor_SMD:R_1206_3216Metric_Pad1.30x1.75mm_HandSolder, F.Cu at (66.4, 255.8)
- added R53: 10K, Resistor_SMD:R_1206_3216Metric_Pad1.30x1.75mm_HandSolder, F.Cu at (89.6, 233.1)
- added R54: 220R, Resistor_SMD:R_1206_3216Metric_Pad1.30x1.75mm_HandSolder, F.Cu at (75.9, 245.5)
- added R55: 2K2, Resistor_SMD:R_1206_3216Metric_Pad1.30x1.75mm_HandSolder, F.Cu at (66.4, 252.5)
- added R56: CREZ12061%, Resistor_SMD:R_1206_3216Metric_Pad1.30x1.75mm_HandSolder, F.Cu at (141.2, 302.7)
- added R57: 510R, Resistor_SMD:R_1206_3216Metric_Pad1.30x1.75mm_HandSolder, F.Cu at (147.1, 299.2)
- added R58: 330R, Resistor_SMD:R_0603_1608Metric_Pad0.98x0.95mm_HandSolder, F.Cu at (152.3, 295.5)
- added R59: 4K7, Resistor_SMD:R_1206_3216Metric_Pad1.30x1.75mm_HandSolder, F.Cu at (127.6, 234.9)
- added R6: 10K, Resistor_SMD:R_1206_3216Metric_Pad1.30x1.75mm_HandSolder, F.Cu at (148.5, 287.4)
- added R60: 4K7, Resistor_SMD:R_1206_3216Metric_Pad1.30x1.75mm_HandSolder, F.Cu at (121.6, 241.5)
- added R7: 10K, Resistor_SMD:R_1206_3216Metric_Pad1.30x1.75mm_HandSolder, F.Cu at (142.5, 284.1)
- added R8: 4K3, Resistor_SMD:R_1206_3216Metric_Pad1.30x1.75mm_HandSolder, F.Cu at (142.5, 287.4)
- added R9: 4K3, Resistor_SMD:R_1206_3216Metric_Pad1.30x1.75mm_HandSolder, F.Cu at (165.1, 263.6)
- added SW1: SPST2P, RetroBitLab:SPST-7.3x3.9x2.5-WUERTH-434121025816, F.Cu at (110.2, 225.9)
- added SW2: SPST_SWITCH_SMD_4P,4.1x5.4mm, RetroBitLab:SW_DIP_SPSTx02_DSHP02TS-S, F.Cu at (67.3, 237.1)
- added U15: L7805, Package_TO_SOT_SMD:TO-252-2, F.Cu at (76.9, 227.3)
- added U5: IC74HC00, Package_SO:SOIC-14_3.9x8.7mm_P1.27mm, F.Cu at (101.4, 228.3)
- added U7: ESP32-PICO-D4, RetroBitLab:ESP32-PICO-D4, F.Cu at (101.9, 238.1)
- added U9: IC74HC00, Package_SO:SOIC-14_3.9x8.7mm_P1.27mm, F.Cu at (54.0, 272.4)
- added Y1: 12MHzC, Crystal:Crystal_SMD_HC49-SD_HandSoldering, F.Cu at (44.1, 226.4)
- C37: value 1uF -> 22uF
- C41: value 22uF -> 22pF
- C43: value 22pF -> 1uF
- C45: value 22pF -> 10uF-20V; footprint Capacitor_SMD:C_1206_3216Metric_Pad1.33x1.80mm_HandSolder -> Capacitor_Tantalum_SMD:CP_EIA-3528-12_Kemet-T_Pad1.50x2.35mm_HandSolder
- D3, D4: value 1N5819 -> DIOSCH20V; footprint Diode_THT:D_DO-41_SOD81_P10.16mm_Horizontal -> Diode_SMD:D_SMC_Handsoldering
- L1: value FB0805/600R/2A -> FB1206100R100MHZ4A; footprint Inductor_SMD:L_0805_2012Metric_Pad1.15x1.40mm_HandSolder -> Inductor_SMD:L_1206_3216Metric_Pad1.42x1.75mm_HandSolder
- Q1, Q2: value BSS138 -> MOSFET-BSS138-SOT-23
- Q3, Q4: value BC817 -> BC817,SOT-23
- U1, U3, U4: value TXB0108DQSR -> TXS0108EPW; footprint Package_SON:USON-20_2x4mm_P0.4mm -> Package_SO:TSSOP-20_4.4x6.5mm_P0.65mm
- U10: footprint Package_SO:SOIC-8_5.23x5.23mm_P1.27mm -> Package_SO:SOIC-8_3.9x4.9mm_P1.27mm
- U12: value AMS1117-3.3 -> USBCH340T; footprint Package_TO_SOT_SMD:SOT-223-3_TabPin2 -> Package_SO:SSOP-20_5.3x7.2mm_P0.65mm
- U13: value TLV71325PDBV -> AMS1117-3.3; footprint Package_TO_SOT_SMD:SOT-23-5 -> Package_TO_SOT_SMD:SOT-223-3_TabPin2
- U14: value CH340T -> AMS1117-2.5; footprint Package_SO:SSOP-20_5.3x7.2mm_P0.65mm -> Package_TO_SOT_SMD:SOT-223-3_TabPin2
- moved C1 194.6 mm to (86.5, 265.5)
- moved C49 188.4 mm to (48.4, 255.3)
- moved U1 187.1 mm to (113.4, 279.8)
- moved C6 186.3 mm to (129.5, 277.5)
- moved C12 185.8 mm to (92.5, 262.1)
- moved X1 185.7 mm to (112.3, 286.5)
- moved C8 183.5 mm to (135.5, 277.5)
- moved U3 183.2 mm to (153.6, 278.5)
- moved C10 183.0 mm to (92.5, 265.5)
- moved C3 181.9 mm to (98.5, 268.9)
- moved C7 181.7 mm to (129.5, 284.2)
- moved C11 181.2 mm to (86.5, 268.9)
- moved C5 180.5 mm to (118.7, 285.5)
- moved U4 177.5 mm to (122.1, 279.8)
- moved Q1 177.3 mm to (146.7, 278.1)
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Connections:
- C1 pad 1: 3V3 -> GND
- C1 pad 2: GND -> 3V3
- C10 pad 1: 5V -> GND
- C10 pad 2: GND -> 5V
- C11 pad 1: 3V3 -> GND
- C11 pad 2: GND -> 3V3
- C12 pad 1: 5V -> GND
- C12 pad 2: GND -> 5V
- C2 pad 1: 5V -> GND
- C2 pad 2: GND -> 5V
- C3 pad 1: 3V3 -> GND
- C3 pad 2: GND -> 3V3
- C37 pad 1: GND -> 5V_USB
- C37 pad 2: 2V5 -> GND
- C38 pad 1: GND -> Net-(C38-Pad1)
- C38 pad 2: 5V -> GND
- C4 pad 1: GND -> 3V3
- C4 pad 2: 3V3 -> GND
- C40 pad 1: GND -> 5V_USB
- C40 pad 2: 3V3 -> GND
- C41 pad 1: GND -> Net-(C41-Pad1)
- C41 pad 2: 5V_USB -> GND
- C42 pad 1: GND -> Net-(C42-Pad1)
- C42 pad 2: Net-(C42-Pad2) -> GND
- C43 pad 1: Net-(C43-Pad1) -> 2V5
- C44 pad 1: GND -> 5V
- C44 pad 2: 5V_USB -> GND
- C45 pad 1: Net-(C45-Pad1) -> 3V3
- C46 pad 1: GND -> 3V3
- C46 pad 2: Net-(C46-Pad2) -> GND
- C49 pad 1: GND -> Net-(C48-Pad1)
- C49 pad 2: Net-(C48-Pad1) -> GND
- C5 pad 1: GND -> 3V3
- C5 pad 2: 3V3 -> GND
- C6 pad 1: GND -> 3V3
- C6 pad 2: 3V3 -> GND
- C7 pad 1: GND -> Net-(C7-Pad1)
- C7 pad 2: Net-(C7-Pad2) -> GND
- C8 pad 1: GND -> Net-(C7-Pad1)
- C8 pad 2: Net-(C7-Pad2) -> GND
- C9 pad 1: 3V3 -> GND
- C9 pad 2: GND -> 3V3
- J4 pad S1: Net-(C46-Pad2) -> Net-(C42-Pad1)
- J4 pad S2: Net-(C46-Pad2) -> Net-(C42-Pad1)
- J4 pad S3: Net-(C46-Pad2) -> Net-(C42-Pad1)
- J4 pad S4: Net-(C46-Pad2) -> Net-(C42-Pad1)
- J4 pad S5: Net-(C46-Pad2) -> Net-(C42-Pad1)
- J4 pad S6: Net-(C46-Pad2) -> Net-(C42-Pad1)
- U1 pad 10: mA4 -> TXB_EN
- U1 pad 11: A4 -> GND
- U1 pad 12: A3 -> A4
- U1 pad 13: A2 -> A3
- U1 pad 14: A1 -> A2
- U1 pad 15: GND -> A1
- U1 pad 16: 5V -> A0
- U1 pad 17: A0 -> ~IRQ
- U1 pad 18: ~IRQ -> ~WE
- U1 pad 19: ~WE -> 5V
- U1 pad 2: ~mWE -> 3V3
- U1 pad 3: ~mVIRQ -> ~mWE
- U1 pad 4: mA0 -> ~mVIRQ
- U1 pad 5: 3V3 -> mA0
- U1 pad 6: Net-(R2-Pad2) -> mA1
- U1 pad 7: mA1 -> mA2
- U1 pad 8: mA2 -> mA3
- U1 pad 9: mA3 -> mA4
- U12 pad 1: GND -> Net-(U12-Pad1)
- U12 pad 2: 3V3 -> Net-(U12-Pad2)
- U12 pad 3: 5V -> Net-(D3-Pad1)
- U13 pad 1: 5V -> GND
- U13 pad 2: GND -> 3V3
- U14 pad 1: Net-(U14-Pad1) -> GND
- U14 pad 2: Net-(U14-Pad2) -> 2V5
- U14 pad 3: Net-(D3-Pad1) -> 5V
- U2 pad 29: Net-(C7-Pad2) -> Net-(C7-Pad1)
- U2 pad 30: Net-(C7-Pad2) -> Net-(C7-Pad1)
- U2 pad 5: Net-(C7-Pad2) -> Net-(C7-Pad1)
- U3 pad 10: mD7 -> TXB_EN
- U3 pad 11: D7 -> GND
- U3 pad 12: D6 -> D7
- U3 pad 13: D5 -> D6
- U3 pad 14: D4 -> D5
- U3 pad 15: GND -> D4
- U3 pad 16: 5V -> D3
- U3 pad 17: D3 -> D2
- U3 pad 18: D2 -> D1
- U3 pad 19: D1 -> 5V
- U3 pad 2: mD1 -> 3V3
- U3 pad 3: mD2 -> mD1
- U3 pad 4: mD3 -> mD2
- U3 pad 5: 3V3 -> mD3
- U3 pad 6: Net-(R6-Pad2) -> mD4
- U3 pad 7: mD4 -> mD5
- U3 pad 8: mD5 -> mD6
- U3 pad 9: mD6 -> mD7
- U4 pad 10: mA8 -> TXB_EN
- U4 pad 11: A8 -> GND
- U4 pad 12: A7 -> A8
- U4 pad 13: A6 -> A7
- U4 pad 14: A5 -> A6
- U4 pad 15: GND -> A5
- U4 pad 16: 5V -> PHI2
- U4 pad 17: PHI2 -> ~MPD
- U4 pad 18: ~MPD -> ~EXSEL
- U4 pad 19: ~EXSEL -> 5V
- U4 pad 2: ~mEXSEL -> 3V3
- U4 pad 3: ~mMPD -> ~mEXSEL
- U4 pad 4: mPHI2 -> ~mMPD
- U4 pad 5: 3V3 -> mPHI2
- U4 pad 6: Net-(R7-Pad2) -> mA5
- U4 pad 7: mA5 -> mA6
- U4 pad 8: mA6 -> mA7
- U4 pad 9: mA7 -> mA8
- U8 pad 11: /Vera FPGA flash/SD_MISO -> /Vera FPGA flash/DAT0
- U8 pad 3: /Vera FPGA flash/SD_CS0 -> /Vera FPGA flash/DAT3
- U8 pad 6: /Vera FPGA flash/SD_MOSI -> /Vera FPGA flash/CMD
- U8 pad 8: /Vera FPGA flash/SD_SCK -> /Vera FPGA flash/CLK
Routing:
- net AUDIO: track 0.00 -> 14.2 mm
- net GND: track 0.00 -> 4.40 mm, vias 0 -> 1
- added copper zone on POWER, net 3V3
- added copper zone on GND, net GND
Other:
- board size 0.9 x 0.6 mm -> 143 x 162 mm
- copper layers 2 -> 4

Commit message: Optimized layout
Parts:
- added C55: 1uF, Capacitor_SMD:C_1206_3216Metric_Pad1.33x1.80mm_HandSolder, B.Cu at (226.3, 195.5)
- added C56: 1uF, Capacitor_SMD:C_1206_3216Metric_Pad1.33x1.80mm_HandSolder, B.Cu at (219.0, 186.3)
- added C57: 1uF, Capacitor_SMD:C_1206_3216Metric_Pad1.33x1.80mm_HandSolder, F.Cu at (276.1, 225.7)
- added C58: 1uF, Capacitor_SMD:C_1206_3216Metric_Pad1.33x1.80mm_HandSolder, F.Cu at (276.1, 229.1)
- added JP3: Jumper3_Bridged12, Jumper:SolderJumper-3_P1.3mm_Open_RoundedPad1.0x1.5mm, F.Cu at (119.2, 113.3)
- added LD5: RED, LED_SMD:LED_1206_3216Metric_Pad1.42x1.75mm_HandSolder, F.Cu at (113.4, 109.8)
- added Q5: MOSFET-BSS138-SOT-23, Package_TO_SOT_SMD:SOT-23, F.Cu at (124.6, 110.4)
- added R61: 330R, Resistor_SMD:R_1206_3216Metric_Pad1.30x1.75mm_HandSolder, F.Cu at (113.4, 113.1)
- added R62: 3K3, Resistor_SMD:R_1206_3216Metric_Pad1.30x1.75mm_HandSolder, F.Cu at (119.4, 109.7)
- added R63: 10K, Resistor_SMD:R_1206_3216Metric_Pad1.30x1.75mm_HandSolder, F.Cu at (113.4, 116.4)
- added R64: 10K, Resistor_SMD:R_1206_3216Metric_Pad1.30x1.75mm_HandSolder, B.Cu at (226.3, 190.0)
- added R65: 0R, Resistor_SMD:R_1206_3216Metric_Pad1.30x1.75mm_HandSolder, F.Cu at (172.0, 49.5)
- added R66: 10K, Resistor_SMD:R_1206_3216Metric_Pad1.30x1.75mm_HandSolder, F.Cu at (276.0, 232.4)
- added TP1: TP5V, TestPoint:TestPoint_Pad_D2.0mm, F.Cu at (172.3, 55.1)
- added U16: TXS0108EPW, Package_SO:TSSOP-20_4.4x6.5mm_P0.65mm, F.Cu at (268.7, 228.1)
- added U17: MAX40200AUK, Package_TO_SOT_SMD:SOT-23-5, F.Cu at (175.7, 58.1)
- added U6: TXS0108EPW, Package_SO:TSSOP-20_4.4x6.5mm_P0.65mm, B.Cu at (220.2, 192.7)
- added mRD4: TestPoint, TestPoint:TestPoint_Pad_D2.0mm, F.Cu at (247.4, 180.4)
- added mRD5: TestPoint, TestPoint:TestPoint_Pad_D2.0mm, F.Cu at (233.2, 165.4)
- added ~mHALT1: TestPoint, TestPoint:TestPoint_Pad_D2.0mm, F.Cu at (239.1, 160.6)
- added ~mRSVD1: TestPoint, TestPoint:TestPoint_Pad_D2.0mm, F.Cu at (224.1, 178.6)
- added ~mS4: TestPoint, TestPoint:TestPoint_Pad_D2.0mm, F.Cu at (243.1, 178.7)
- added ~mS5: TestPoint, TestPoint:TestPoint_Pad_D2.0mm, F.Cu at (254.8, 180.1)
- C1, C2, R2, U1: moved to B.Cu
- R56: value CREZ12061% -> 0R
- moved R56 235.7 mm to (136.0, 67.0), turned to 90 degrees
- moved LD3 226.4 mm to (136.0, 73.0), turned to 90 degrees
- moved R57 224.3 mm to (141.0, 75.0), turned to 180 degrees
- moved R58 220.5 mm to (153.0, 75.0), turned to 90 degrees
- moved LD4 216.2 mm to (152.0, 80.0), turned to 270 degrees
- moved C40 210.7 mm to (161.1, 59.0)
- moved C37 209.5 mm to (155.0, 60.5), turned to 180 degrees
- moved R51 208.6 mm to (156.5, 56.5), turned to 180 degrees
- moved U12 208.5 mm to (162.1, 66.0), turned to 270 degrees
- moved D3 207.3 mm to (171.3, 88.6)
- moved C47 206.9 mm to (141.0, 65.0), turned to 180 degrees
- moved C49 206.0 mm to (148.0, 75.0)
- moved C38 201.3 mm to (169.0, 61.0)
- moved J5 201.1 mm to (147.0, 59.0), turned to 270 degrees
- moved J4 200.7 mm to (160.5, 52.5), turned to 180 degrees
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Connections:
- net Net-(ECI1-Pad6) renamed ~REF
- C1 pad 2: 3V3 -> +3V3
- C10 pad 2: 5V -> +5V
- C11 pad 2: 3V3 -> +3V3
- C12 pad 2: 5V -> +5V
- C2 pad 2: 5V -> +5V
- C3 pad 2: 3V3 -> +3V3
- C4 pad 1: 3V3 -> +3V3
- C5 pad 1: 3V3 -> +3V3
- C6 pad 1: 3V3 -> +3V3
- C9 pad 2: 3V3 -> +3V3
- CART1 pad 1: Net-(CART1-Pad1) -> ~S4
- CART1 pad 12: Net-(CART1-Pad12) -> ~S5
- CART1 pad 14: Net-(CART1-Pad14) -> RD5
- CART1 pad A: Net-(CART1-PadA) -> RD4
- ECI1 pad 3: Net-(ECI1-Pad3) -> ~D1XX
- ECI1 pad A: Net-(ECI1-PadA) -> RSRVD
- ECI1 pad C: Net-(ECI1-PadC) -> ~HALT
- J1 pad 9: 5V -> +5V
- J2 pad 9: 5V -> +5V
- LD2 pad 2: 3V3 -> +3V3
- R2 pad 1: 3V3 -> +3V3
- R5 pad 1: 3V3 -> +3V3
- R56 pad 1: 5V -> Net-(R56-Pad1)
- R6 pad 1: 3V3 -> +3V3
- R7 pad 1: 3V3 -> +3V3
- SW2 pad 4: TBX_EN -> TXB_EN
- U1 pad 1: ~mRE -> mD2
- U1 pad 12: A4 -> ~S4
- U1 pad 17: ~IRQ -> D4
- U1 pad 18: ~WE -> D5
- U1 pad 19: 5V -> +5V
- U1 pad 2: 3V3 -> +3V3
- U1 pad 20: ~RE -> D2
- U1 pad 3: ~mWE -> mD5
- U1 pad 4: ~mVIRQ -> mD4
- U1 pad 9: mA4 -> ~mS4
- U2 pad 1: 3V3 -> +3V3
- U2 pad 22: 3V3 -> +3V3
- U2 pad 33: 3V3 -> +3V3
- U3 pad 1: mD0 -> mRD4
- U3 pad 12: D7 -> A12
- U3 pad 13: D6 -> A9
- U3 pad 14: D5 -> A8
- U3 pad 15: D4 -> A7
- U3 pad 16: D3 -> A6
- U3 pad 17: D2 -> A5
- U3 pad 18: D1 -> A4
- U3 pad 19: 5V -> +5V
- U3 pad 2: 3V3 -> +3V3
- U3 pad 20: D0 -> RD4
- U3 pad 3: mD1 -> mA4
- U3 pad 4: mD2 -> mA5
- U3 pad 5: mD3 -> mA6
- U3 pad 6: mD4 -> mA7
- U3 pad 7: mD5 -> mA8
- U3 pad 8: mD6 -> mA9
- U3 pad 9: mD7 -> mA12
- U4 pad 1: ~FPGA_RESET -> mD3
- U4 pad 12: A8 -> ~IRQ
- U4 pad 13: A7 -> RSRVD
- U4 pad 14: A6 -> PHI2
- U4 pad 15: A5 -> R~W
- U4 pad 16: PHI2 -> A10
- U4 pad 17: ~MPD -> A11
- U4 pad 18: ~EXSEL -> D7
- U4 pad 19: 5V -> +5V
- U4 pad 2: 3V3 -> +3V3
- U4 pad 20: ~RST -> D3
- U4 pad 3: ~mEXSEL -> mD7
- U4 pad 4: ~mMPD -> mA11
- U4 pad 5: mPHI2 -> mA10
- U4 pad 6: mA5 -> mR~W
- U4 pad 7: mA6 -> mPHI2
- U4 pad 8: mA7 -> mRSRVD
- U4 pad 9: mA8 -> ~mVIRQ
- X1 pad 4: 3V3 -> +3V3
Routing:
- net RSRVD: track 0.00 -> 64.6 mm, vias 0 -> 2
- net ~IRQ: track 0.00 -> 64.1 mm
- net ~EXSEL: track 0.00 -> 61.8 mm
- net ~RST: track 0.00 -> 61.8 mm
- net +5V: track 0.00 -> 39.9 mm, vias 0 -> 6
- net PHI2: track 0.00 -> 39.0 mm, vias 0 -> 2
- net +3V3: track 0.00 -> 38.7 mm, vias 0 -> 6
- net R~W: track 0.00 -> 32.1 mm
- net A12: track 0.00 -> 23.5 mm
- net A9: track 0.00 -> 22.9 mm
- net 5V: track 0.00 -> 21.9 mm, vias 0 -> 2
- net A8: track 0.00 -> 21.0 mm
- net A10: track 0.00 -> 20.6 mm
- net ~CCTL: track 0.00 -> 20.1 mm
- net A7: track 0.00 -> 18.9 mm
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Other:
- rule pad_to_mask_clearance: 0 -> 0.1

Commit message: Some placements
Parts:
- C13, C14, C58: moved to B.Cu
- moved C19 191.6 mm to (212.6, 142.9), turned to 90 degrees
- moved C13 188.0 mm to (213.7, 141.1), turned to 180 degrees
- moved C20 186.9 mm to (215.1, 142.9), turned to 90 degrees
- moved C21 185.4 mm to (222.1, 141.9)
- moved C14 179.2 mm to (213.7, 144.4), turned to 180 degrees
- moved C15 178.5 mm to (207.8, 152.1), turned to 270 degrees
- moved C22 177.2 mm to (222.1, 144.5)
- moved C16 173.7 mm to (210.3, 152.1), turned to 270 degrees
- moved C23 173.5 mm to (216.2, 163.0)
- moved C24 170.3 mm to (216.2, 159.4)
- moved C17 167.4 mm to (197.6, 152.0), turned to 270 degrees
- moved C18 162.8 mm to (200.2, 152.0), turned to 270 degrees
- moved R66 118.0 mm to (168.5, 183.8), turned to 180 degrees
- moved L1 116.3 mm to (204.1, 150.7)
- moved C58 114.6 mm to (168.2, 190.5)
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Routing:
- net ~RE: track 13.1 -> 78.1 mm, vias 0 -> 2
- net ~WE: track 6.33 -> 64.5 mm, vias 0 -> 2
- net 3V3: track 0.00 -> 51.9 mm, vias 0 -> 5
- net GND: track 22.9 -> 57.0 mm, vias 7 -> 15
- net ~D1XX: track 0.00 -> 23.1 mm, vias 0 -> 1
- net AUDIO: track 0.00 -> 20.5 mm, vias 0 -> 2
- net ~MPD: track 0.00 -> 14.4 mm, vias 0 -> 1
- net ~HALT: track 0.00 -> 13.6 mm
- net A13: track 0.00 -> 13.1 mm
- net A14: track 0.00 -> 13.0 mm, vias 0 -> 2
- net A15: track 0.00 -> 12.0 mm, vias 0 -> 2
- net Net-(C15-Pad1): track 0.00 -> 9.60 mm
- net +5V: track 39.9 -> 45.9 mm, vias 6 -> 7
- net TXB_EN: track 8.26 -> 13.2 mm
- net 5V: track 21.9 -> 26.2 mm, vias 2 -> 3

Commit message: Optimized layout
Parts:
- C53, C54, R29, R30: moved to B.Cu
- moved C54 254.0 mm to (217.5, 54.9)
- moved R30 238.1 mm to (202.8, 52.4), turned to 180 degrees
- moved R29 234.7 mm to (208.3, 52.4), turned to 180 degrees
- moved R13 221.1 mm to (199.5, 69.0), turned to 180 degrees
- moved R28 220.3 mm to (193.0, 76.2), turned to 180 degrees
- moved R22 218.4 mm to (193.0, 72.5), turned to 180 degrees
- moved R19 216.4 mm to (199.5, 72.5), turned to 180 degrees
- moved R10 215.8 mm to (187.5, 65.2), turned to 180 degrees
- moved R27 212.7 mm to (187.5, 76.2), turned to 180 degrees
- moved R21 211.8 mm to (187.5, 72.5), turned to 180 degrees
- moved R16 206.2 mm to (193.0, 68.9), turned to 180 degrees
- moved R14 205.1 mm to (205.0, 69.0), turned to 180 degrees
- moved C53 201.4 mm to (195.3, 54.5), turned to 180 degrees
- moved R9 201.0 mm to (199.5, 65.5), turned to 180 degrees
- moved R15 195.3 mm to (187.5, 68.9), turned to 180 degrees
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Routing:
- net ~RE: track 78.1 -> 13.1 mm, vias 2 -> 0
- net RSRVD: track 64.6 -> 0.00 mm, vias 2 -> 0
- net ~IRQ: track 64.1 -> 0.00 mm
- net ~EXSEL: track 61.8 -> 0.00 mm
- net ~RST: track 61.8 -> 0.00 mm
- net ~WE: track 64.5 -> 6.33 mm, vias 2 -> 0
- net PHI2: track 39.0 -> 8.37 mm
- net A12: track 23.5 -> 0.00 mm
- net ~D1XX: track 23.1 -> 0.00 mm, vias 1 -> 0
- net A9: track 22.9 -> 0.00 mm
- net R~W: track 32.1 -> 9.31 mm
- net A8: track 21.0 -> 0.00 mm
- net A10: track 20.6 -> 0.00 mm
- net ~CCTL: track 20.1 -> 0.00 mm
- net A7: track 18.9 -> 0.00 mm
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Other:
- board size 143 x 162 mm -> 143 x 162.5 mm

Commit message: Updated
Parts:
- moved C3 230.0 mm to (217.6, 72.0)
- moved JP1 230.0 mm to (249.0, 102.6)
- moved R25 230.0 mm to (260.5, 84.0)
- moved X1 230.0 mm to (231.4, 89.7)
- moved R20 230.0 mm to (255.7, 90.6)
- moved R49 230.0 mm to (266.2, 99.1)
- moved R8 230.0 mm to (261.6, 90.6)
- moved C5 230.0 mm to (237.8, 88.7)
- moved C6 230.0 mm to (248.6, 80.7)
- moved C7 230.0 mm to (248.6, 87.4)
- moved C8 230.0 mm to (254.6, 80.7)
- moved LD2 230.0 mm to (243.8, 90.7)
- moved R5 230.0 mm to (254.6, 87.3)
- moved U2 205.6 mm to (208.5, 84.3)
- moved C26 185.7 mm to (155.3, 124.3)
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Routing:
- net ~IRQ: track 0.00 -> 62.2 mm
- net RSRVD: track 0.00 -> 61.6 mm
- net R~W: track 9.31 -> 54.5 mm, vias 0 -> 2
- net PHI2: track 8.37 -> 51.6 mm, vias 2 -> 3
- net ~RE: track 13.1 -> 44.8 mm, vias 0 -> 1
- net ~D1XX: track 0.00 -> 27.9 mm, vias 0 -> 2
- net A12: track 0.00 -> 27.8 mm
- net A9: track 0.00 -> 27.1 mm
- net A10: track 0.00 -> 26.7 mm
- net ~MPD: track 0.00 -> 26.6 mm, vias 0 -> 2
- net A8: track 0.00 -> 26.3 mm
- net A11: track 0.00 -> 25.9 mm
- net ~CCTL: track 0.00 -> 25.9 mm
- net A7: track 0.00 -> 25.5 mm
- net D7: track 0.00 -> 25.1 mm
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
Commit message: Updated
Parts:
- moved ~mS5 31.2 mm to (220.4, 165.7)
Connections:
- net ~REF renamed Net-(ECI1-Pad6)
Routing:
- net ~EXSEL: track 0.00 -> 60.8 mm, vias 0 -> 2
- net ~RST: track 0.00 -> 58.6 mm, vias 0 -> 2
- net ~WE: track 6.33 -> 55.7 mm, vias 0 -> 4
- net mRD5: track 0.00 -> 22.4 mm, vias 0 -> 2
- net ~mS4: track 0.00 -> 15.6 mm, vias 0 -> 1
- net ~RE: track 44.8 -> 59.7 mm, vias 1 -> 2
- net ~mS5: track 0.00 -> 14.6 mm, vias 0 -> 1
- net mRSRVD: track 2.07 -> 15.5 mm
- net mRD4: track 0.00 -> 12.3 mm
- net 5V: track 23.2 -> 29.9 mm, vias 2 -> 3
- net GND: track 62.0 -> 67.0 mm, vias 18 -> 19
- net RSRVD: track 61.6 -> 65.6 mm
- net ~IRQ: track 62.2 -> 64.6 mm

Commit message: Updated
Parts:
- moved R26 77.7 mm to (211.1, 75.9), turned to 180 degrees
- moved R23 75.6 mm to (219.9, 75.8), turned to 180 degrees
- moved R12 74.6 mm to (225.4, 68.6), turned to 180 degrees
- moved R18 73.0 mm to (225.5, 72.1), turned to 180 degrees
- moved R24 72.3 mm to (225.5, 75.8), turned to 180 degrees
- moved R17 68.9 mm to (219.9, 72.1), turned to 180 degrees
- moved R11 65.8 mm to (219.9, 68.6), turned to 180 degrees
- moved R25 55.5 mm to (205.6, 75.9), turned to 180 degrees
- moved R8 48.9 mm to (219.9, 65.1), turned to 180 degrees
- moved R20 48.2 mm to (211.1, 72.2), turned to 180 degrees
- moved C3 13.5 mm to (216.7, 85.5)
- moved R13 6.11 mm to (205.6, 68.7)
- moved R14 6.11 mm to (211.1, 68.7)
- moved R19 6.11 mm to (205.6, 72.2)
- moved R9 6.11 mm to (205.6, 65.2)
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Other:
- board text added: "BLUE"
- board text added: "GREEN"
- board text added: "RED"

Commit message: Updated
Parts:
- added C59: 1uF, Capacitor_SMD:C_1206_3216Metric_Pad1.33x1.80mm_HandSolder, B.Cu at (205.9, 93.2)
- added C60: 1uF, Capacitor_SMD:C_1206_3216Metric_Pad1.33x1.80mm_HandSolder, B.Cu at (211.7, 93.2)
- C3, C31, C6, C7, R45: moved to B.Cu
- U14: value AMS1117-2.5 -> AMS1117-1.5
- U2: footprint Package_DFN_QFN:QFN-48-1EP_7x7mm_P0.5mm_EP5.6x5.6mm -> RetroBitLab:QFN-48-1EP_7x7mm_P0.5mm_EP5.6x5.6mm
- moved J3 121.6 mm to (250.0, 56.2), turned to 180 degrees
- moved Q1 100.3 mm to (179.3, 51.6), turned to 90 degrees
- moved U9 94.9 mm to (226.9, 54.0)
- moved JP2 92.8 mm to (235.4, 50.0), turned to 270 degrees
- moved U10 92.2 mm to (235.4, 59.8)
- moved R1 87.0 mm to (183.9, 49.4), turned to 180 degrees
- moved U11 85.0 mm to (223.1, 82.4)
- moved J1 83.1 mm to (250.9, 74.8), turned to 90 degrees
- moved C31 82.4 mm to (235.4, 80.0)
- moved R46 74.1 mm to (230.2, 80.0), turned to 180 degrees
- moved LD2 70.7 mm to (183.9, 53.1), turned to 180 degrees
- moved C30 68.3 mm to (235.4, 80.0)
- moved R45 67.3 mm to (230.1, 79.9), turned to 180 degrees
- moved C7 45.8 mm to (203.3, 80.5), turned to 180 degrees
- moved JP3 44.7 mm to (228.7, 102.3)
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Connections:
- C3 pad 2: +3V3 -> 3V3
- C4 pad 1: +3V3 -> 3V3
- C43 pad 1: 2V5 -> 1V5
- C5 pad 1: +3V3 -> 3V3
- C51 pad 1: 2V5 -> 1V5
- C6 pad 1: +3V3 -> 3V3
- C7 pad 1: Net-(C7-Pad1) -> 1V5
- C8 pad 1: Net-(C7-Pad1) -> 1V5
- J1 pad 11: Net-(J1-Pad11) -> AUDIOL
- J1 pad 12: Net-(J1-Pad12) -> AUDIOR
- J1 pad 15: Net-(J1-Pad15) -> 5V
- J1 pad 16: Net-(J1-Pad16) -> 3V3
- J1 pad 4: Net-(J1-Pad4) -> 3V3
- J1 pad 9: +5V -> 5V
- R5 pad 1: +3V3 -> 3V3
- U14 pad 2: 2V5 -> 1V5
- U2 pad 1: +3V3 -> 3V3
- U2 pad 22: +3V3 -> 3V3
- U2 pad 24: 2V5 -> 3V3
- U2 pad 29: Net-(C7-Pad1) -> 1V5
- U2 pad 30: Net-(C7-Pad1) -> 1V5
- U2 pad 33: +3V3 -> 3V3
- U2 pad 44: /VeraModule/VGA_VSYNC -> /VeraModule/VGA_HSYNC
- U2 pad 45: /VeraModule/VGA_HSYNC -> /VeraModule/VGA_VSYNC
- U2 pad 5: Net-(C7-Pad1) -> 1V5
- X1 pad 4: +3V3 -> 3V3
Routing:
- net FPGA_CDONE: track 0.00 -> 128.7 mm, vias 0 -> 2
- net mD2: track 0.00 -> 68.3 mm
- net /VeraModule/VGA_R3: track 0.00 -> 57.3 mm
- net /VeraModule/VGA_R2: track 0.00 -> 50.6 mm
- net /VeraModule/VGA_HSYNC: track 0.00 -> 50.2 mm, vias 0 -> 1
- net /VeraModule/VGA_R1: track 0.00 -> 44.5 mm
- net /VeraModule/VGA_VSYNC: track 0.00 -> 42.3 mm, vias 0 -> 1
- net 3V3: track 51.9 -> 88.7 mm, vias 5 -> 14
- net /VeraModule/VGA_R0: track 0.00 -> 35.8 mm
- net GND: track 67.0 -> 93.6 mm, vias 19 -> 26
- net /VeraModule/VGA_B0: track 0.00 -> 25.8 mm
- net /VeraModule/VGA_B1: track 0.00 -> 21.8 mm
- net /VeraModule/VGA_G0: track 0.00 -> 18.7 mm
- net 1V5: track 0.00 -> 18.3 mm, vias 0 -> 2
- net /VeraModule/VGA_B2: track 0.00 -> 17.7 mm
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- removed copper zone on POWER, net 3V3
- removed copper zone on GND, net GND
